File: 02_Boards/01_Energex8PCB_v1.0/01_Energex8PCB_v1.0.kicad_pcb (KiCad board)
At the start: 4 copper layers, 205 x 92 mm, 107 parts, among them J1 XT60-M, J10 XT60-M, J11 61300211121, J12 B2B-PH-K-S, J13 XT60-M, J14 61300211121, J15 B2B-PH-K-S, J16 XT60-M, J17 61300211121, J18 B2B-PH-K-S, J19 XT60-M, J2 XT60-M, J20 61300211121, J21 B2B-PH-K-S, J22 XT60-M, J23 61300211121, J24 B2B-PH-K-S, J25 XT60-M, J26 61300211121, J27 B2B-PH-K-S, J28 XT60-M, J29 61300211121, J3 XT60-M, J30 B2B-PH-K-S, J31 XT60-M, J32 B2B-PH-K-S, J33 B2B-PH-K-S, J34 B2B-PH-K-S, J35 B2B-PH-K-S, J36 B2B-PH-K-S, J37 B2B-PH-K-S, J38 B2B-PH-K-S, J39 B2B-PH-K-S, J4 B2B-PH-K-S, J5 B2B-PH-K-S, J6 XT60-M, J7 XT60-M, J8 61300211121, J9 B2B-PH-K-S, U1 0986AH0304, U10 0986AH0304, U11 0986AH0304, U12 0986AH0304, U2 0986AH0304, U3 0986AH0304, U4 0986AH0304, U5 0986AH0304, U6 0986AH0304, U7 0986AH0304, U8 0986AH0304, U9 0986AH0304

Commit message: PCB Documentation
Parts:
- moved G*** 2.54 mm to (203.1, 174.0)
- moved G*** 2.54 mm to (246.3, 172.8)
Changed lines of the file:
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@@
 			(outputformat 1)
 			(mirror no)
-			(drillshape 1)
+			(drillshape 0)
 			(scaleselection 1)
-			(outputdirectory "")
+			(outputdirectory "02_Board_Outputs/01_Board_Blueprints/")
 		)
 	)
@@
 	(footprint "01_Footprints:EA7LAULogo2_UserDrawings"
 		(layer "F.Cu")
-		(at 243.713 172.847)
+		(at 246.253 172.847)
 		(property "Reference" "G***"
 			(at 0 0 0)
@@
 	(footprint "01_Footprints:Energex8Logo_UserDrawings"
 		(layer "F.Cu")
-		(at 200.533 173.99)
+		(at 203.073 173.99)
 		(property "Reference" "G***"
 			(at 0 0 0)
@@
 		)
 	)
+	(dimension
+		(type orthogonal)
+		(layer "Cmts.User")
+		(pts
+			(xy 46.538 134.244) (xy 251.538 134.244)
+		)
+		(height 13.584)
+		(orientation 0)
+		(format
+			(prefix "")
+			(suffix "")
+			(units 3)
+			(units_format 1)
+			(precision 2)
+		)
+		(style
+			(thickness 0.15)
+			(arrow_length 1.27)
+			(text_position_mode 0)
+			(arrow_direction outward)
+			(extension_height 0.58642)
+			(extension_offset 0.5)
+			(keep_text_aligned yes)
+		)
+		(gr_text "205.00 mm"
+			(at 149.038 146.028 0)
+			(layer "Cmts.User")
+			(effects
+				(font
+					(size 1.5 1.5)
+					(thickness 0.3)
+					(bold yes)
+				)
+			)
+		)
+	)
+	(dimension
+		(type orthogonal)
+		(layer "Cmts.User")
+		(pts
+			(xy 246.38 47.244) (xy 246.538 139.244)
+		)
+		(height 14.224)
+		(orientation 1)
+		(format
+			(prefix "")
+			(suffix "")
+			(units 3)
+			(units_format 1)
+			(precision 2)
+		)
+		(style
+			(thickness 0.15)
+			(arrow_length 1.27)
+			(text_position_mode 0)
+			(arrow_direction outward)
+			(extension_height 0.58642)
+			(extension_offset 0.5)
+			(keep_text_aligned yes)
+		)
+		(gr_text "92.00 mm"
+			(at 258.804 93.244 90)
+			(layer "Cmts.User")
+			(effects
+				(font
+					(size 1.5 1.5)
+					(thickness 0.3)
+					(bold yes)
+				)
+			)
+		)
+	)

Commit message: Relative routes
Parts:
- renumbered H3 to H2, H4 to H3
