File: 02_Boards/01_Energex8PCB_v1.0/01_Energex8PCB_v1.0.kicad_sch (KiCad schematic)
At the start: 104 parts, among them J1 XT60-M, J10 XT60-M, J11 61300211121, J12 B2B-PH-K-S, J13 XT60-M, J14 61300211121, J15 B2B-PH-K-S, J16 XT60-M, J17 61300211121, J18 B2B-PH-K-S, J19 XT60-M, J2 XT60-M, J20 61300211121, J21 B2B-PH-K-S, J22 XT60-M, J23 61300211121, J24 B2B-PH-K-S, J25 XT60-M, J26 61300211121, J27 B2B-PH-K-S, J28 XT60-M, J29 61300211121, J3 XT60-M, J30 B2B-PH-K-S, J31 XT60-M, J32 B2B-PH-K-S, J33 B2B-PH-K-S, J34 B2B-PH-K-S, J35 B2B-PH-K-S, J36 B2B-PH-K-S, J37 B2B-PH-K-S, J38 B2B-PH-K-S, J39 B2B-PH-K-S, J4 B2B-PH-K-S, J5 B2B-PH-K-S, J6 XT60-M, J7 XT60-M, J8 61300211121, J9 B2B-PH-K-S, U1 0986AH0304, U10 0986AH0304, U11 0986AH0304, U12 0986AH0304, U2 0986AH0304, U3 0986AH0304, U4 0986AH0304, U5 0986AH0304, U6 0986AH0304, U7 0986AH0304, U8 0986AH0304, U9 0986AH0304

Commit message: PCB Documentation
Changed lines of the file:
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@@
 	(symbol
 		(lib_id "EA7LAULogo2:LOGO")
-		(at 243.84 172.72 0)
+		(at 246.38 172.72 0)
 		(unit 1)
 		(exclude_from_sim no)
@@
 		(fields_autoplaced yes)
 		(property "Reference" "#G2"
-			(at 243.84 148.3458 0)
+			(at 246.38 148.3458 0)
 			(effects
 				(font
@@
 		)
 		(property "Value" "LOGO"
-			(at 243.84 197.0942 0)
+			(at 246.38 197.0942 0)
 			(effects
 				(font
@@
 		)
 		(property "Footprint" ""
-			(at 243.84 172.72 0)
+			(at 246.38 172.72 0)
 			(effects
 				(font
@@
 		)
 		(property "Datasheet" ""
-			(at 243.84 172.72 0)
+			(at 246.38 172.72 0)
 			(effects
 				(font
@@
 		)
 		(property "Description" ""
-			(at 243.84 172.72 0)
+			(at 246.38 172.72 0)
 			(effects
 				(font
@@
 	(symbol
 		(lib_id "Energex8Logo:LOGO")
-		(at 200.66 173.99 0)
+		(at 203.2 173.99 0)
 		(unit 1)
 		(exclude_from_sim no)
@@
 		(fields_autoplaced yes)
 		(property "Reference" "#G1"
-			(at 200.66 149.6158 0)
+			(at 203.2 149.6158 0)
 			(effects
 				(font
@@
 		)
 		(property "Value" "LOGO"
-			(at 200.66 198.3642 0)
+			(at 203.2 198.3642 0)
 			(effects
 				(font
@@
 		)
 		(property "Footprint" ""
-			(at 200.66 173.99 0)
+			(at 203.2 173.99 0)
 			(effects
 				(font
@@
 		)
 		(property "Datasheet" ""
-			(at 200.66 173.99 0)
+			(at 203.2 173.99 0)
 			(effects
 				(font
@@
 		)
 		(property "Description" ""
-			(at 200.66 173.99 0)
+			(at 203.2 173.99 0)
 			(effects
 				(font

Commit message: Relative routes
Parts:
- removed H2: MountingHole_Pad, MountingHole:MountingHole_3.2mm_M3_Pad_Via, symbol Mechanical:MountingHole_Pad
- J1, J2, J3, J6, J7: Description_1 (none) -> Plug; DC supply; XT60; male; PIN: 2; for cable; soldered; 3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
- renumbered H3 to H2, H4 to H3
Other:
- moved on the sheet: H1, H2, H3
